File: KiCAD/SPECTACOAL_KiCAD/SPECTACOAL/SPECTACOAL.kicad_sch (KiCad schematic)
At the start: 13 parts, among them SW1 Reset, U1 TiVa, U2 Joystick_2_Axis_1SW, U3 Joystick_2_Axis_1SW

Commit message: add buttons
Parts:
- added R3: 10k, symbol ME218_BaseLib:Res1
- added SW2: Reset, symbol ME218_BaseLib:SW-PB
Connections:
- net +3.3V: now also SW2.1
- net GNDREF: now also R3.1
- net at SPECTACOAL1.12 (RA4): now also R3.2, SW2.2
Changed lines of the file:
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@@
   (junction (at 82.55 104.14) (diameter 0) (color 0 0 0 0)
   )
+  (junction (at 46.99 77.47) (diameter 0) (color 0 0 0 0)
+  )
   (junction (at 68.58 49.53) (diameter 0) (color 0 0 0 0)
   )
@@
   )
   (wire (pts (xy 124.46 81.28) (xy 107.95 81.28))
+    (stroke (width 0) (type default))
+  )
+  (wire (pts (xy 46.99 77.47) (xy 68.58 77.47))
     (stroke (width 0) (type default))
   )
@@
     )
   )
+  (symbol (lib_id "ME218_BaseLib:Res1") (at 46.99 81.28 180) (unit 1)
+    (in_bom yes) (on_board yes) (dnp no)
+    (property "Reference" "R3" (at 40.64 81.28 90)
+      (effects (font (size 1.27 1.27)) hide)
+    )
+    (property "Value" "10k" (at 49.53 81.28 90)
+      (effects (font (size 1.27 1.27)))
+    )
+    (property "Footprint" "" (at 45.974 81.026 90)
+      (effects (font (size 1.27 1.27)) hide)
+    )
+    (property "Datasheet" "" (at 46.99 81.28 0)
+      (effects (font (size 1.27 1.27)) hide)
+    )
+    (pin "1")
+    (pin "2")
+    (instances
+      (project "SPECTACOAL"
+        (path "/7b7f6bb2-7e9a-4004-b852-742946769482"
+          (reference "R3") (unit 1)
+        )
+      )
+      (project "218CProjectKiCad"
+        (path "/90de9929-b4af-488b-8896-c9a198ebb96b"
+          (reference "R4") (unit 1)
+        )
+      )
+    )
+  )
   (symbol (lib_id "ME218_BaseLib:Motor_Servo") (at 109.22 123.19 0) (unit 1)
     (in_bom yes) (on_board yes) (dnp no) (fields_autoplaced)
@@
         (path "/90de9929-b4af-488b-8896-c9a198ebb96b"
           (reference "#PWR034") (unit 1)
+        )
+      )
+    )
+  )
+  (symbol (lib_id "power:GNDREF") (at 46.99 85.09 0) (unit 1)
+    (in_bom yes) (on_board yes) (dnp no) (fields_autoplaced)
+    (property "Reference" "#PWR018" (at 46.99 91.44 0)
+      (effects (font (size 1.27 1.27)) hide)
+    )
+    (property "Value" "GNDREF" (at 46.99 90.17 0)
+      (effects (font (size 1.27 1.27)))
+    )
+    (property "Footprint" "" (at 46.99 85.09 0)
+      (effects (font (size 1.27 1.27)) hide)
+    )
+    (property "Datasheet" "" (at 46.99 85.09 0)
+      (effects (font (size 1.27 1.27)) hide)
+    )
+    (pin "1")
+    (instances
+      (project "SPECTACOAL"
+        (path "/7b7f6bb2-7e9a-4004-b852-742946769482"
+          (reference "#PWR018") (unit 1)
+        )
+      )
+      (project "218CProjectKiCad"
+        (path "/90de9929-b4af-488b-8896-c9a198ebb96b"
+          (reference "#PWR015") (unit 1)
         )
       )
@@
     )
   )
+  (symbol (lib_id "power:+3.3V") (at 46.99 67.31 0) (unit 1)
+    (in_bom yes) (on_board yes) (dnp no) (fields_autoplaced)
+    (property "Reference" "#PWR017" (at 46.99 71.12 0)
+      (effects (font (size 1.27 1.27)) hide)
+    )
+    (property "Value" "+3.3V" (at 46.99 62.23 0)
+      (effects (font (size 1.27 1.27)))
+    )
+    (property "Footprint" "" (at 46.99 67.31 0)
+      (effects (font (size 1.27 1.27)) hide)
+    )
+    (property "Datasheet" "" (at 46.99 67.31 0)
+      (effects (font (size 1.27 1.27)) hide)
+    )
+    (pin "1")
+    (instances
+      (project "SPECTACOAL"
+        (path "/7b7f6bb2-7e9a-4004-b852-742946769482"
+          (reference "#PWR017") (unit 1)
+        )
+      )
+      (project "218CProjectKiCad"
+        (path "/90de9929-b4af-488b-8896-c9a198ebb96b"
+          (reference "#PWR033") (unit 1)
+        )
+      )
+    )
+  )
   (symbol (lib_id "power:GNDREF") (at 101.6 125.73 0) (unit 1)
     (in_bom yes) (on_board yes) (dnp no) (fields_autoplaced)
@@
         )
       )
+    )
+  )
+  (symbol (lib_id "ME218_BaseLib:SW-PB") (at 46.99 72.39 90) (mirror x) (unit 1)
+    (in_bom yes) (on_board yes) (dnp no)
+    (property "Reference" "SW2" (at 43.18 71.12 90)
+      (effects (font (size 1.27 1.27)) (justify left))
+    )
+    (property "Value" "Reset" (at 43.18 73.66 90)
+      (effects (font (size 1.27 1.27)) (justify left))
+    )
+    (property "Footprint" "" (at 41.91 72.39 0)
+      (effects (font (size 1.27 1.27)) hide)
+    )
+    (property "Datasheet" "" (at 41.91 72.39 0)
+      (effects (font (size 1.27 1.27)) hide)
+    )
+    (pin "1")
+    (pin "2")
+    (instances
+      (project "SPECTACOAL"
+        (path "/7b7f6bb2-7e9a-4004-b852-742946769482"
+          (reference "SW2") (unit 1)
+        )
+      )
+      (project "218CProjectKiCad"
+        (path "/90de9929-b4af-488b-8896-c9a198ebb96b"
+          (reference "SW2") (unit 1)
+        )
+      )
