File: KiCAD/SPECTACOAL_KiCAD/SPECTACOAL/SPECTACOAL.kicad_sch (KiCad schematic)
At the start: 22 parts, among them SW1 Reset, SW2 Reset, U1 TiVa, U2 Joystick_2_Axis_1SW, U3 Joystick_2_Axis_1SW, U4 D168K

Commit message: update KiCAD for report
Parts:
- added D3: pairing indicator, symbol ME218_BaseLib:LED
- added R8: 47Ohm, symbol ME218_BaseLib:Res1
- added U5: LSM6DS33 IMU, LSM6DS33:PQFN50P300X300X86-16N, symbol LSM6DS33:LSM6DS33
Connections:
- net +3.3V: now also U5.1 (VDD), U5.2 (VIN)
- net +5V: now also U1.1 (VCC)
- net CS for IMU: now also SPECTACOAL1.10 (RA3); no longer SPECTACOAL1.3 (RA1)
- net GND: now also R8.2, U5.3 (GND); no longer SPECTACOAL1.12 (RA4)
- net QH: now also D3.2 (A)
- net U2RX: now also U1.2 (DOUT)
- net U2TX: now also U1.3 (DIN)
- net at R3.1, SW2.1: now also SPECTACOAL1.12 (RA4)
- net MISO/SDI renamed SPI MISO for IMU
- net MOSI/SDO renamed SPI MOSI for IMU
- net SPI SCK renamed SPI SCK for IMU
- net Tera renamed Serial Debug
- new net: D3.1 (K), R8.1
- new net RA3 of PIC32: U5.7 (CS)
- new net RCLK: SPECTACOAL1.3 (RA1)
- new net SPI MISO from PIC32: U5.6 (SDO)
- new net SPI MOSI from PIC32: U5.4 (SDA)
- new net SPI SCK from PIC32: U5.5 (SCL)
- no-connect marks 0 -> 19
Other:
- moved on the sheet: C1, C2, C3, C4, Charge_Indicator, PRG1, R1, R2, SPECTACOAL1, SW1, SW2, U1A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
