File: KiCAD/SPECTACOAL_KiCAD/SPECTACOAL/_autosave-SPECTACOAL.kicad_sch (KiCad schematic)
At the start: 15 parts, among them SW1 Reset, SW2 Reset, U1 TiVa, U2 Joystick_2_Axis_1SW, U3 Joystick_2_Axis_1SW

Commit message: update
Parts:
- added D1: LED-charging indicator, symbol ME218_BaseLib:LED
- added D2: LED-drive mode indicator, symbol ME218_BaseLib:LED
- added R4, R5: 47Ohm, symbol ME218_BaseLib:Res1
- added R6, R7: R_pull, symbol ME218_BaseLib:Res1
- added U4: D168K, Display_7Segment:D1X8K, symbol Display_Character:D168K
- R3: value 10k -> R_pull
Connections:
- net +3.3V: now also R3.2, R6.2, R7.2; no longer SW2.1
- net GND: now also C1.2, C2.2, C3.1, C4.2, Charge_Indicator.3 (-), SPECTACOAL1.12 (RA4), SPECTACOAL1.19 (Vss), SPECTACOAL1.27 (AVss), SPECTACOAL1.8 (Vss), SW1.2, SW2.2, U1.10 (GND), U2.1 (GND), U3.1 (GND), R4.2, R5.2, U4.3 (CC), U4.8 (CC)
- net SER shift_reg: no longer SPECTACOAL1.9 (RA2)
- net at SPECTACOAL1.11 (RB4), U2.5 (SW): now also R7.1
- net at SPECTACOAL1.18 (PGED2/5VT/RB9), U3.5 (SW): now also R6.1
- net at SPECTACOAL1.6 (RB2): now also D1.2 (A)
- net at SPECTACOAL1.7 (RB3): now also D2.2 (A)
- removed net GNDREF: C1.2, C2.2, C3.1, C4.2, Charge_Indicator.3 (-), R3.1, SPECTACOAL1.19 (Vss), SPECTACOAL1.27 (AVss), SPECTACOAL1.8 (Vss), SW1.2, U1.10 (GND), U2.1 (GND), U3.1 (GND)
- net RCLK shift_reg renamed RCLK
- net SRCLK shift_reg renamed SRCLK
- new net: D1.1 (K), R4.1
- new net: D2.1 (K), R5.1
- new net: R3.1, SW2.1
- new net QA: U4.7 (A)
- new net QB: U4.6 (B)
- new net QC: U4.4 (C)
- new net QD: U4.2 (D)
- new net QE: U4.1 (E)
- new net QF: U4.9 (F)
- new net QG: U4.10 (G)
- new net SER: SPECTACOAL1.9 (RA2)
Other:
- note added: "SN74HC595 shift register"
- moved on the sheet: C1, C2, C3, C4, Charge_Indicator, PRG1, R1, R2, SPECTACOAL1, SW1, SW2, U1A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
